File: key-pcb.kicad_pcb (KiCad board)
At the start: 2 copper layers, 14.2 x 14.2 mm, 16 parts

Commit message: V2
Parts:
- + (x2), - (x2), IN (x2), OUT (x2), c (x2), r (x2): footprint TestPoint:TestPoint_Pad_1.0x1.0mm -> Library:TestPoint_Pad_1.5x1.5mm_with_hole
- moved + 15.0 mm to (143.5, 102.2)
- moved - 12.1 mm to (132.0, 91.0)
- moved - 11.5 mm to (143.6, 91.0)
- moved c 9.22 mm to (134.8, 91.1)
- moved D 6.47 mm to (141.2, 95.3), turned to -90 degrees
- moved OUT 1.95 mm to (143.6, 96.6)
- moved IN 1.90 mm to (132.0, 96.6)
- moved c 1.35 mm to (141.3, 99.1)
- moved IN 1.19 mm to (143.6, 99.4)
- moved OUT 1.10 mm to (132.0, 99.4)
- moved r 0.83 mm to (143.6, 93.8)
- moved r 0.70 mm to (132.0, 93.8)
- moved cap 0.66 mm to (134.9, 97.8)
- moved + 0.30 mm to (132.0, 102.2)
Routing:
- net VSS: track 29.3 -> 45.2 mm, vias 8 -> 4
- net VDD: track 22.4 -> 15.5 mm, vias 3 -> 1
- net Net-(D1-A): track 2.63 -> 9.01 mm
- net /col: track 10.3 -> 14.6 mm, vias 2 -> 1
- net /row: track 16.4 -> 12.5 mm
- net /DOUT: track 17.3 -> 18.1 mm
- net /DIN: track 15.7 -> 15.8 mm, vias 2 -> 1
- removed copper zone on B.Cu, net VSS
