File: rgbmain.kicad_sch (KiCad schematic)
At the start: 15 parts, among them J1 Conn_01x10_Pin, J10 Conn_01x04, J2 Conn_01x10_Pin, J3 Conn_01x09_Pin, J4 Conn_01x09, J5 Conn_01x06_Pin, J6 Conn_01x06, J7 Conn_01x13, J8 Conn_01x13, J9 Conn_01x01, Q1 BSS138, U1 Elite-Pi

Commit message: pcb layout complete
Parts:
- renumbered J8 to J1, J7 to J2, J6 to J3, J5 to J4, J4 to J5, J3 to J6, J2 to J7, J1 to J8
Connections:
- net SLC0 is gone; now on net SCL0: J10.4 (Pin_4)
- net VDD is gone; now on net +5V: J5.4 (Pin_4), J6.6 (Pin_6), J7.10 (Pin_10), J8.10 (Pin_10)
- net VSS is gone; now on net GND: J5.1 (Pin_1), J6.9 (Pin_9), J7.9 (Pin_9), J8.9 (Pin_9)
Changed lines of the file:
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@@
 	(wire
 		(pts
+			(xy 78.74 68.58) (xy 82.55 68.58)
+		)
+		(stroke
+			(width 0)
+			(type default)
+		)
+	)
+	(wire
+		(pts
 			(xy 113.03 31.75) (xy 118.11 31.75)
 		)
@@
 	(wire
 		(pts
+			(xy 78.74 63.5) (xy 82.55 63.5)
+		)
+		(stroke
+			(width 0)
+			(type default)
+		)
+	)
+	(wire
+		(pts
 			(xy 243.84 69.85) (xy 246.38 69.85)
 		)
@@
 		)
 	)
-	(label "SLC0"
+	(label "SCL0"
 		(at 113.03 34.29 180)
 		(effects
@@
 		)
 	)
+	(label "VDD"
+		(at 82.55 63.5 0)
+		(effects
+			(font
+				(size 1.27 1.27)
+			)
+			(justify left bottom)
+		)
+	)
 	(label "COL_7"
 		(at 247.65 30.48 0)
@@
 		)
 	)
+	(label "VSS"
+		(at 82.55 68.58 0)
+		(effects
+			(font
+				(size 1.27 1.27)
+			)
+			(justify left bottom)
+		)
+	)
 	(label "ROW_4"
 		(at 30.48 113.03 180)
@@
 		(on_board yes)
 		(dnp no)
-		(property "Reference" "J7"
+		(property "Reference" "J2"
 			(at 38.1 19.05 0)
 			(effects
@@
 			(project ""
 				(path "/24ca604d-a7a4-46c7-a288-45b7cfc45cc9"
-					(reference "J7")
+					(reference "J2")
 					(unit 1)
 				)
@@
 		(dnp no)
 		(fields_autoplaced yes)
-		(property "Reference" "J6"
-			(at 236.22 72.3899 0)
+		(property "Reference" "J3"
+			(at 238.76 60.96 0)
 			(effects
 				(font
 					(size 1.27 1.27)
 				)
-				(justify left)
 			)
 		)
 		(property "Value" "Conn_01x06"
-			(at 236.22 74.9299 0)
+			(at 238.76 63.5 0)
 			(effects
 				(font
 					(size 1.27 1.27)
 				)
-				(justify left)
 			)
 		)
@@
 			(project ""
 				(path "/24ca604d-a7a4-46c7-a288-45b7cfc45cc9"
-					(reference "J6")
+					(reference "J3")
 					(unit 1)
 				)
@@
 		(on_board yes)
 		(dnp no)
-		(property "Reference" "J2"
+		(property "Reference" "J7"
 			(at 152.146 162.814 0)
 			(effects
@@
 			(project ""
 				(path "/24ca604d-a7a4-46c7-a288-45b7cfc45cc9"
-					(reference "J2")
+					(reference "J7")
 					(unit 1)
 				)
@@
 		(on_board yes)
 		(dnp no)
-		(property "Reference" "J5"
+		(property "Reference" "J4"
 			(at 40.64 74.9301 0)
 			(effects
@@
 			(project ""
 				(path "/24ca604d-a7a4-46c7-a288-45b7cfc45cc9"
-					(reference "J5")
+					(reference "J4")
 					(unit 1)
 				)
@@
 		(on_board yes)
 		(dnp no)
-		(property "Reference" "J1"
+		(property "Reference" "J8"
 			(at 124.968 160.02 0)
 			(effects
@@
 			(project ""
 				(path "/24ca604d-a7a4-46c7-a288-45b7cfc45cc9"
-					(reference "J1")
+					(reference "J8")
 					(unit 1)
 				)
@@
 		(dnp no)
 		(fields_autoplaced yes)
-		(property "Reference" "J4"
-			(at 236.22 104.1399 0)
+		(property "Reference" "J5"
+			(at 238.76 88.9 0)
 			(effects
 				(font
 					(size 1.27 1.27)
 				)
-				(justify left)
 			)
 		)
 		(property "Value" "Conn_01x09"
-			(at 236.22 106.6799 0)
+			(at 238.76 91.44 0)
 			(effects
 				(font
 					(size 1.27 1.27)
 				)
-				(justify left)
 			)
 		)
@@
 			(project ""
 				(path "/24ca604d-a7a4-46c7-a288-45b7cfc45cc9"
-					(reference "J4")
+					(reference "J5")
 					(unit 1)
 				)
@@
 		(on_board yes)
 		(dnp no)
-		(property "Reference" "J3"
+		(property "Reference" "J6"
 			(at 38.1 88.9 0)
 			(effects
@@
 			(project ""
 				(path "/24ca604d-a7a4-46c7-a288-45b7cfc45cc9"
-					(reference "J3")
+					(reference "J6")
+					(unit 1)
+				)
+			)
+		)
+	)
+	(symbol
+		(lib_id "power:+5V")
+		(at 78.74 63.5 0)
+		(unit 1)
+		(exclude_from_sim no)
+		(in_bom yes)
+		(on_board yes)
+		(dnp no)
+		(fields_autoplaced yes)
+		(property "Reference" "#PWR010"
+			(at 78.74 67.31 0)
+			(effects
+				(font
+					(size 1.27 1.27)
+				)
+				(hide yes)
+			)
+		)
+		(property "Value" "+5V"
+			(at 78.74 58.42 0)
+			(effects
+				(font
+					(size 1.27 1.27)
+				)
+			)
+		)
+		(property "Footprint" ""
+			(at 78.74 63.5 0)
+			(effects
+				(font
+					(size 1.27 1.27)
+				)
+				(hide yes)
+			)
+		)
+		(property "Datasheet" ""
+			(at 78.74 63.5 0)
+			(effects
+				(font
+					(size 1.27 1.27)
+				)
+				(hide yes)
+			)
+		)
+		(property "Description" "Power symbol creates a global label with name \"+5V\""
+			(at 78.74 63.5 0)
+			(effects
+				(font
+					(size 1.27 1.27)
+				)
+				(hide yes)
+			)
+		)
+		(pin "1"
+		)
+		(instances
+			(project ""
+				(path "/24ca604d-a7a4-46c7-a288-45b7cfc45cc9"
+					(reference "#PWR010")
 					(unit 1)
 				)
@@
 		(dnp no)
 		(fields_autoplaced yes)
-		(property "Reference" "J8"
-			(at 236.22 39.3699 0)
+		(property "Reference" "J1"
+			(at 238.76 19.05 0)
 			(effects
 				(font
 					(size 1.27 1.27)
 				)
-				(justify left)
 			)
 		)
 		(property "Value" "Conn_01x13"
-			(at 236.22 41.9099 0)
+			(at 238.76 21.59 0)
 			(effects
 				(font
 					(size 1.27 1.27)
 				)
-				(justify left)
 			)
 		)
@@
 			(project ""
 				(path "/24ca604d-a7a4-46c7-a288-45b7cfc45cc9"
-					(reference "J8")
+					(reference "J1")
 					(unit 1)
 				)
@@
 					(unit 1)
 				)
+			)
+		)
+	)
+	(symbol
+		(lib_id "power:GND")
+		(at 78.74 68.58 0)
+		(unit 1)
+		(exclude_from_sim no)
+		(in_bom yes)
+		(on_board yes)
+		(dnp no)
+		(fields_autoplaced yes)
+		(property "Reference" "#PWR09"
+			(at 78.74 74.93 0)
+			(effects
+				(font
+					(size 1.27 1.27)
+				)
+				(hide yes)
+			)
+		)
+		(property "Value" "GND"
+			(at 78.74 73.66 0)
+			(effects
+				(font
+					(size 1.27 1.27)
+				)
+			)
+		)
+		(property "Footprint" ""
+			(at 78.74 68.58 0)
+			(effects
+				(font
+					(size 1.27 1.27)
+				)
+				(hide yes)
+			)
+		)
+		(property "Datasheet" ""
+			(at 78.74 68.58 0)
+			(effects
+				(font
+					(size 1.27 1.27)
+				)
+				(hide yes)
+			)
+		)
+		(property "Description" "Power symbol creates a global label with name \"GND\" , ground"
+			(at 78.74 68.58 0)
+			(effects
+				(font
+					(size 1.27 1.27)
+				)
+				(hide yes)
+			)
+		)
+		(pin "1"
+		)
+		(instances
+			(project ""
+				(path "/24ca604d-a7a4-46c7-a288-45b7cfc45cc9"
+					(reference "#PWR09")
+					(unit 1)
+				)

Commit message: changed thumb connectors
wanted thumbs to be the same as stock.
Parts:
- J7, J8: footprint Connector_Molex:Molex_KK-254_AE-6410-10A_1x10_P2.54mm_Vertical -> Connector_PinHeader_2.54mm:PinHeader_1x10_P2.54mm_Vertical
Changed lines of the file:
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@@
 			)
 		)
-		(property "Footprint" "Connector_Molex:Molex_KK-254_AE-6410-10A_1x10_P2.54mm_Vertical"
+		(property "Footprint" "Connector_PinHeader_2.54mm:PinHeader_1x10_P2.54mm_Vertical"
 			(at 161.29 144.78 0)
 			(effects
@@
 			)
 		)
-		(property "Footprint" "Connector_Molex:Molex_KK-254_AE-6410-10A_1x10_P2.54mm_Vertical"
+		(property "Footprint" "Connector_PinHeader_2.54mm:PinHeader_1x10_P2.54mm_Vertical"
 			(at 128.27 144.78 0)
 			(effects
