File: thumb-pcb/kinesis-thumb-pcb.kicad_sch (KiCad schematic)
At the start: 50 parts, among them J1 Conn_01x10, J2 Conn_01x10

Commit message: Part placement
Parts:
- J2: footprint Pin_Headers:Pin_Header_Straight_1x10_Pitch2.54mm -> Connector_PinHeader_2.54mm:PinHeader_1x10_P2.54mm_Vertical
- renumbered C6 to C25, C5 to C35, C3 to C36, C2 to C46, C4 to C55, C1 to C56, C12 to C65, C9 to C66, C11 to C75, C10 to C85, C8 to C86, C7 to C96, D6 to D25, D5 to D35, D3 to D36, D2 to D46, D4 to D55, D1 to D56, D12 to D65, D9 to D66, D11 to D75, D10 to D85, D8 to D86, D7 to D96
Other:
- company: dcpedit -> fritz - (orginal dcpedit)
- title: PillzMod thumb cluster PCB -> rgbkin thumb cluster PCB
Changed lines of the file:
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@@
 	(paper "A4")
 	(title_block
-		(title "PillzMod thumb cluster PCB")
-		(date "2024-03-13")
-		(rev "1")
-		(company "dcpedit")
+		(title "rgbkin thumb cluster PCB")
+		(date "2025-08-30")
+		(rev "2")
+		(company "fritz - (orginal dcpedit)")
 	)
 	(junction
@@
 		(on_board yes)
 		(dnp no)
-		(property "Reference" "D2"
+		(property "Reference" "D46"
 			(at 38.2016 62.3316 90)
 			(effects
@@
 			(project "kinesis-thumb-pcb"
 				(path "/c801d42e-dd94-493e-bd2f-6c3ddad43f55"
-					(reference "D2")
+					(reference "D46")
 					(unit 1)
 				)
@@
 		(on_board yes)
 		(dnp no)
-		(property "Reference" "D1"
+		(property "Reference" "D56"
 			(at 38.2016 42.6466 90)
 			(effects
@@
 			(project "kinesis-thumb-pcb"
 				(path "/c801d42e-dd94-493e-bd2f-6c3ddad43f55"
-					(reference "D1")
+					(reference "D56")
 					(unit 1)
 				)
@@
 		(dnp no)
 		(fields_autoplaced yes)
-		(property "Reference" "C12"
+		(property "Reference" "C65"
 			(at 240.03 127.0062 0)
 			(effects
@@
 			(project "kinesis-thumb-pcb"
 				(path "/c801d42e-dd94-493e-bd2f-6c3ddad43f55"
-					(reference "C12")
+					(reference "C65")
 					(unit 1)
 				)
@@
 		(dnp no)
 		(fields_autoplaced yes)
-		(property "Reference" "C2"
+		(property "Reference" "C46"
 			(at 96.52 63.5062 0)
 			(effects
@@
 			(project ""
 				(path "/c801d42e-dd94-493e-bd2f-6c3ddad43f55"
-					(reference "C2")
+					(reference "C46")
 					(unit 1)
 				)
@@
 		(on_board yes)
 		(dnp no)
-		(property "Reference" "D8"
+		(property "Reference" "D86"
 			(at 162.6616 62.3316 90)
 			(effects
@@
 			(project "kinesis-thumb-pcb"
 				(path "/c801d42e-dd94-493e-bd2f-6c3ddad43f55"
-					(reference "D8")
+					(reference "D86")
 					(unit 1)
 				)
@@
 		(dnp no)
 		(fields_autoplaced yes)
-		(property "Reference" "C1"
+		(property "Reference" "C56"
 			(at 96.52 33.0262 0)
 			(effects
@@
 			(project ""
 				(path "/c801d42e-dd94-493e-bd2f-6c3ddad43f55"
-					(reference "C1")
+					(reference "C56")
 					(unit 1)
 				)
@@
 		(on_board yes)
 		(dnp no)
-		(property "Reference" "D10"
+		(property "Reference" "D85"
 			(at 177.2666 62.3316 90)
 			(effects
@@
 			(project "kinesis-thumb-pcb"
 				(path "/c801d42e-dd94-493e-bd2f-6c3ddad43f55"
-					(reference "D10")
+					(reference "D85")
 					(unit 1)
 				)
@@
 		(on_board yes)
 		(dnp no)
-		(property "Reference" "D12"
+		(property "Reference" "D65"
 			(at 177.2666 101.7016 90)
 			(effects
@@
 			(project "kinesis-thumb-pcb"
 				(path "/c801d42e-dd94-493e-bd2f-6c3ddad43f55"
-					(reference "D12")
+					(reference "D65")
 					(unit 1)
 				)
@@
 		(dnp no)
 		(fields_autoplaced yes)
-		(property "Reference" "C11"
+		(property "Reference" "C75"
 			(at 240.03 93.9862 0)
 			(effects
@@
 			(project "kinesis-thumb-pcb"
 				(path "/c801d42e-dd94-493e-bd2f-6c3ddad43f55"
-					(reference "C11")
+					(reference "C75")
 					(unit 1)
 				)
@@
 		(on_board yes)
 		(dnp no)
-		(property "Reference" "D7"
+		(property "Reference" "D96"
 			(at 162.6616 42.6466 90)
 			(effects
@@
 			(project "kinesis-thumb-pcb"
 				(path "/c801d42e-dd94-493e-bd2f-6c3ddad43f55"
-					(reference "D7")
+					(reference "D96")
 					(unit 1)
 				)
@@
 		(on_board yes)
 		(dnp no)
-		(property "Reference" "D6"
+		(property "Reference" "D25"
 			(at 52.8066 101.7016 90)
 			(effects
@@
 			(project "kinesis-thumb-pcb"
 				(path "/c801d42e-dd94-493e-bd2f-6c3ddad43f55"
-					(reference "D6")
+					(reference "D25")
 					(unit 1)
 				)
@@
 		(on_board yes)
 		(dnp no)
-		(property "Reference" "D5"
+		(property "Reference" "D35"
 			(at 52.8066 82.0166 90)
 			(effects
@@
 			(project "kinesis-thumb-pcb"
 				(path "/c801d42e-dd94-493e-bd2f-6c3ddad43f55"
-					(reference "D5")
+					(reference "D35")
 					(unit 1)
 				)
@@
 		(dnp no)
 		(fields_autoplaced yes)
-		(property "Reference" "C7"
+		(property "Reference" "C96"
 			(at 224.79 33.0262 0)
 			(effects
@@
 			(project "kinesis-thumb-pcb"
 				(path "/c801d42e-dd94-493e-bd2f-6c3ddad43f55"
-					(reference "C7")
+					(reference "C96")
 					(unit 1)
 				)
@@
 		(dnp no)
 		(fields_autoplaced yes)
-		(property "Reference" "C5"
+		(property "Reference" "C35"
 			(at 111.76 93.9862 0)
 			(effects
@@
 			(project ""
 				(path "/c801d42e-dd94-493e-bd2f-6c3ddad43f55"
-					(reference "C5")
+					(reference "C35")
 					(unit 1)
 				)
@@
 		(on_board yes)
 		(dnp no)
-		(property "Reference" "D3"
+		(property "Reference" "D36"
 			(at 38.2016 82.0166 90)
 			(effects
@@
 			(project "kinesis-thumb-pcb"
 				(path "/c801d42e-dd94-493e-bd2f-6c3ddad43f55"
-					(reference "D3")
+					(reference "D36")
 					(unit 1)
 				)
@@
 		(on_board yes)
 		(dnp no)
-		(property "Reference" "D11"
+		(property "Reference" "D75"
 			(at 177.2666 82.0166 90)
 			(effects
@@
 			(project "kinesis-thumb-pcb"
 				(path "/c801d42e-dd94-493e-bd2f-6c3ddad43f55"
-					(reference "D11")
+					(reference "D75")
 					(unit 1)
 				)
@@
 		(dnp no)
 		(fields_autoplaced yes)
-		(property "Reference" "C4"
+		(property "Reference" "C55"
 			(at 111.76 33.0262 0)
 			(effects
@@
 			(project "kinesis-thumb-pcb"
 				(path "/c801d42e-dd94-493e-bd2f-6c3ddad43f55"
-					(reference "C4")
+					(reference "C55")
 					(unit 1)
 				)
@@
 			)
 		)
-		(property "Footprint" "Pin_Headers:Pin_Header_Straight_1x10_Pitch2.54mm"
+		(property "Footprint" "Connector_PinHeader_2.54mm:PinHeader_1x10_P2.54mm_Vertical"
 			(at 91.44 167.64 0)
 			(effects
@@
 		(dnp no)
 		(fields_autoplaced yes)
-		(property "Reference" "C9"
+		(property "Reference" "C66"
 			(at 224.79 127.0062 0)
 			(effects
@@
 			(project "kinesis-thumb-pcb"
 				(path "/c801d42e-dd94-493e-bd2f-6c3ddad43f55"
-					(reference "C9")
+					(reference "C66")
 					(unit 1)
 				)
@@
 		(on_board yes)
 		(dnp no)
-		(property "Reference" "D9"
+		(property "Reference" "D66"
 			(at 162.6616 101.7016 90)
 			(effects
@@
 			(project "kinesis-thumb-pcb"
 				(path "/c801d42e-dd94-493e-bd2f-6c3ddad43f55"
-					(reference "D9")
+					(reference "D66")
 					(unit 1)
 				)
@@
 		(on_board yes)
 		(dnp no)
-		(property "Reference" "D4"
+		(property "Reference" "D55"
 			(at 52.8066 42.6466 90)
 			(effects
@@
 			(project "kinesis-thumb-pcb"
 				(path "/c801d42e-dd94-493e-bd2f-6c3ddad43f55"
-					(reference "D4")
+					(reference "D55")
 					(unit 1)
 				)
@@
 		(dnp no)
 		(fields_autoplaced yes)
-		(property "Reference" "C8"
+		(property "Reference" "C86"
 			(at 224.79 63.5062 0)
 			(effects
@@
 			(project "kinesis-thumb-pcb"
 				(path "/c801d42e-dd94-493e-bd2f-6c3ddad43f55"
-					(reference "C8")
+					(reference "C86")
 					(unit 1)
 				)
@@
 		(dnp no)
 		(fields_autoplaced yes)
-		(property "Reference" "C6"
+		(property "Reference" "C25"
 			(at 111.76 127.0062 0)
 			(effects
@@
 			(project ""
 				(path "/c801d42e-dd94-493e-bd2f-6c3ddad43f55"
-					(reference "C6")
+					(reference "C25")
 					(unit 1)
 				)
@@
 		(dnp no)
 		(fields_autoplaced yes)
-		(property "Reference" "C3"
+		(property "Reference" "C36"
 			(at 96.52 93.9862 0)
 			(effects
@@
 			(project ""
 				(path "/c801d42e-dd94-493e-bd2f-6c3ddad43f55"
-					(reference "C3")
+					(reference "C36")
 					(unit 1)
 				)
@@
 		(dnp no)
 		(fields_autoplaced yes)
-		(property "Reference" "C10"
+		(property "Reference" "C85"
 			(at 240.03 63.5062 0)
 			(effects
@@
 			(project "kinesis-thumb-pcb"
 				(path "/c801d42e-dd94-493e-bd2f-6c3ddad43f55"
-					(reference "C10")
+					(reference "C85")
 					(unit 1)
 				)

Commit message: SOD123 Diodes
Parts:
- C25, C35, C36, C46, C55, C56, C65, C66, C75, C85, C86, C96: value C_Small -> 0.1 µF
Changed lines of the file:
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@@
 			)
 		)
-		(property "Value" "C_Small"
+		(property "Value" "0.1 µF"
 			(at 240.03 129.5462 0)
 			(effects
@@
 			)
 		)
-		(property "Value" "C_Small"
+		(property "Value" "0.1 µF"
 			(at 96.52 66.0462 0)
 			(effects
@@
 			)
 		)
-		(property "Value" "C_Small"
+		(property "Value" "0.1 µF"
 			(at 96.52 35.5662 0)
 			(effects
@@
 			)
 		)
-		(property "Value" "C_Small"
+		(property "Value" "0.1 µF"
 			(at 240.03 96.5262 0)
 			(effects
@@
 			)
 		)
-		(property "Value" "C_Small"
+		(property "Value" "0.1 µF"
 			(at 224.79 35.5662 0)
 			(effects
@@
 			)
 		)
-		(property "Value" "C_Small"
+		(property "Value" "0.1 µF"
 			(at 111.76 96.5262 0)
 			(effects
@@
 			)
 		)
-		(property "Value" "C_Small"
+		(property "Value" "0.1 µF"
 			(at 111.76 35.5662 0)
 			(effects
@@
 			)
 		)
-		(property "Value" "C_Small"
+		(property "Value" "0.1 µF"
 			(at 224.79 129.5462 0)
 			(effects
@@
 			)
 		)
-		(property "Value" "C_Small"
+		(property "Value" "0.1 µF"
 			(at 224.79 66.0462 0)
 			(effects
@@
 			)
 		)
-		(property "Value" "C_Small"
+		(property "Value" "0.1 µF"
 			(at 111.76 129.5462 0)
 			(effects
@@
 			)
 		)
-		(property "Value" "C_Small"
+		(property "Value" "0.1 µF"
 			(at 96.52 96.5262 0)
 			(effects
@@
 			)
 		)
-		(property "Value" "C_Small"
+		(property "Value" "0.1 µF"
 			(at 240.03 66.0462 0)
 			(effects

Commit message: Routed
Parts:
- removed J2: Conn_01x10, Connector_PinHeader_2.54mm:PinHeader_1x10_P2.54mm_Vertical, symbol kicad_port-rescue:Conn_01x10-Connector_Generic
Connections:
- net DOUT_L is gone; now on net COL_R6: J1.7 (Pin_7), LED55.2 (DOUT)
- net ROW_2 is gone; now on net DOUT_R: D25.1 (K), J1.2 (Pin_2)
- net ROW_3 is gone; now on net COL_R5: D35.1 (K), D36.1 (K), J1.8 (Pin_8)
- net ROW_4 is gone; now on net DIN_R: D46.1 (K), J1.1 (Pin_1)
- net ROW_6 is gone; now on net ROW_5: D65.1 (K), D66.1 (K)
- net ROW_7 is gone; now on net COL_L6: D75.1 (K)
- net ROW_8 is gone; now on net COL_L5: D85.1 (K), D86.1 (K)
- net ROW_9 is gone; now on net DIN_L: D96.1 (K)
Changed lines of the file:
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@@
 	(wire
 		(pts
-			(xy 96.52 160.02) (xy 105.41 160.02)
-		)
-		(stroke
-			(width 0)
-			(type default)
-		)
-	)
-	(wire
-		(pts
 			(xy 109.22 30.48) (xy 109.22 31.75)
 		)
@@
 	(wire
 		(pts
-			(xy 96.52 180.34) (xy 105.41 180.34)
+			(xy 71.12 177.8) (xy 105.41 177.8)
 		)
 		(stroke
@@
 	(wire
 		(pts
-			(xy 96.52 165.1) (xy 105.41 165.1)
+			(xy 209.55 20.32) (xy 209.55 22.86)
 		)
 		(stroke
@@
 	(wire
 		(pts
-			(xy 209.55 20.32) (xy 209.55 22.86)
+			(xy 88.9 60.96) (xy 93.98 60.96)
 		)
 		(stroke
@@
 	(wire
 		(pts
-			(xy 88.9 60.96) (xy 93.98 60.96)
+			(xy 237.49 114.3) (xy 237.49 124.46)
 		)
 		(stroke
@@
 	(wire
 		(pts
-			(xy 237.49 114.3) (xy 237.49 124.46)
+			(xy 71.12 172.72) (xy 105.41 172.72)
 		)
 		(stroke
@@
 	(wire
 		(pts
+			(xy 71.12 167.64) (xy 105.41 167.64)
+		)
+		(stroke
+			(width 0)
+			(type default)
+		)
+	)
+	(wire
+		(pts
 			(xy 237.49 50.8) (xy 237.49 60.96)
 		)
@@
 	(wire
 		(pts
-			(xy 254 20.32) (xy 254 53.34)
+			(xy 71.12 157.48) (xy 105.41 157.48)
 		)
 		(stroke
@@
 	(wire
 		(pts
-			(xy 96.52 172.72) (xy 105.41 172.72)
+			(xy 254 20.32) (xy 254 53.34)
 		)
 		(stroke
@@
 	(wire
 		(pts
-			(xy 96.52 177.8) (xy 105.41 177.8)
+			(xy 73.66 91.44) (xy 73.66 147.32)
 		)
 		(stroke
@@
 	(wire
 		(pts
-			(xy 73.66 91.44) (xy 73.66 147.32)
+			(xy 93.98 50.8) (xy 93.98 60.96)
 		)
 		(stroke
@@
 	(wire
 		(pts
-			(xy 93.98 50.8) (xy 93.98 60.96)
+			(xy 222.25 30.48) (xy 222.25 31.75)
 		)
 		(stroke
@@
 	(wire
 		(pts
-			(xy 96.52 170.18) (xy 105.41 170.18)
+			(xy 237.49 124.46) (xy 237.49 125.73)
 		)
 		(stroke
@@
 	(wire
 		(pts
-			(xy 222.25 30.48) (xy 222.25 31.75)
+			(xy 71.12 162.56) (xy 105.41 162.56)
 		)
 		(stroke
@@
 	(wire
 		(pts
-			(xy 237.49 124.46) (xy 237.49 125.73)
+			(xy 118.11 91.44) (xy 109.22 91.44)
 		)
 		(stroke
@@
 	(wire
 		(pts
-			(xy 118.11 91.44) (xy 109.22 91.44)
+			(xy 71.12 165.1) (xy 105.41 165.1)
 		)
 		(stroke
@@
 	(wire
 		(pts
-			(xy 156.21 86.995) (xy 175.26 86.995)
+			(xy 71.12 180.34) (xy 105.41 180.34)
 		)
 		(stroke
@@
 	(wire
 		(pts
-			(xy 96.52 167.64) (xy 105.41 167.64)
+			(xy 156.21 86.995) (xy 175.26 86.995)
 		)
 		(stroke
@@
 	(wire
 		(pts
+			(xy 71.12 175.26) (xy 105.41 175.26)
+		)
+		(stroke
+			(width 0)
+			(type default)
+		)
+	)
+	(wire
+		(pts
 			(xy 36.195 86.995) (xy 50.8 86.995)
 		)
@@
 	(wire
 		(pts
-			(xy 133.35 147.32) (xy 133.35 151.13)
+			(xy 71.12 170.18) (xy 105.41 170.18)
 		)
 		(stroke
@@
 	(wire
 		(pts
-			(xy 109.22 81.28) (xy 109.22 91.44)
+			(xy 133.35 147.32) (xy 133.35 151.13)
 		)
 		(stroke
@@
 	(wire
 		(pts
-			(xy 109.22 97.79) (xy 109.22 100.33)
+			(xy 109.22 81.28) (xy 109.22 91.44)
 		)
 		(stroke
@@
 	(wire
 		(pts
-			(xy 246.38 124.46) (xy 237.49 124.46)
+			(xy 109.22 97.79) (xy 109.22 100.33)
 		)
 		(stroke
@@
 	(wire
 		(pts
-			(xy 217.17 30.48) (xy 222.25 30.48)
+			(xy 246.38 124.46) (xy 237.49 124.46)
 		)
 		(stroke
@@
 	(wire
 		(pts
-			(xy 217.17 60.96) (xy 222.25 60.96)
+			(xy 217.17 30.48) (xy 222.25 30.48)
 		)
 		(stroke
@@
 	(wire
 		(pts
-			(xy 118.11 30.48) (xy 109.22 30.48)
+			(xy 217.17 60.96) (xy 222.25 60.96)
 		)
 		(stroke
@@
 	(wire
 		(pts
-			(xy 96.52 175.26) (xy 105.41 175.26)
+			(xy 118.11 30.48) (xy 109.22 30.48)
 		)
 		(stroke
@@
 	(wire
 		(pts
-			(xy 96.52 162.56) (xy 105.41 162.56)
+			(xy 254 68.58) (xy 254 83.82)
 		)
 		(stroke
@@
 	(wire
 		(pts
-			(xy 254 68.58) (xy 254 83.82)
+			(xy 246.38 60.96) (xy 237.49 60.96)
 		)
 		(stroke
@@
 	(wire
 		(pts
-			(xy 246.38 60.96) (xy 237.49 60.96)
+			(xy 71.12 160.02) (xy 105.41 160.02)
 		)
 		(stroke
@@
 	(wire
 		(pts
-			(xy 96.52 157.48) (xy 105.41 157.48)
-		)
-		(stroke
-			(width 0)
-			(type default)
-		)
-	)
-	(wire
-		(pts
 			(xy 93.98 81.28) (xy 93.98 91.44)
 		)
@@
 					(unit 1)
 				)
-			)
-		)
-	)
-	(symbol
-		(lib_id "kicad_port-rescue:Conn_01x10-Connector_Generic")
-		(at 91.44 167.64 0)
-		(mirror y)
-		(unit 1)
-		(exclude_from_sim no)
-		(in_bom yes)
-		(on_board yes)
-		(dnp no)
-		(property "Reference" "J2"
-			(at 88.2904 169.0116 90)
-			(effects
-				(font
-					(size 1.27 1.27)
-				)
-			)
-		)
-		(property "Value" "Conn_01x10"
-			(at 85.979 169.0116 90)
-			(effects
-				(font
-					(size 1.27 1.27)
-				)
-			)
-		)
-		(property "Footprint" "Connector_PinHeader_2.54mm:PinHeader_1x10_P2.54mm_Vertical"
-			(at 91.44 167.64 0)
-			(effects
-				(font
-					(size 1.27 1.27)
-				)
-				(hide yes)
-			)
-		)
-		(property "Datasheet" "~"
-			(at 91.44 167.64 0)
-			(effects
-				(font
-					(size 1.27 1.27)
-				)
-				(hide yes)
-			)
-		)
-		(property "Description" ""
-			(at 91.44 167.64 0)
-			(effects
-				(font
-					(size 1.27 1.27)
-				)
-			)
-		)
-		(pin "1"
-		)
-		(pin "10"
-		)
-		(pin "2"
-		)
-		(pin "3"
-		)
-		(pin "4"
-		)
-		(pin "5"
-		)
-		(pin "6"
-		)
-		(pin "7"
-		)
-		(pin "8"
-		)
-		(pin "9"
-		)
-		(instances
-			(project "kinesis-thumb-pcb"
-				(path "/c801d42e-dd94-493e-bd2f-6c3ddad43f55"
-					(reference "J2")
-					(unit 1)
-				)
