File: thumb-pcb/kinesis-thumb-pcb.kicad_pcb (KiCad board)
At the start: 2 copper layers, 77 x 88 mm, 33 parts, among them J1 Conn_01x10

Commit message: Part placement
Parts:
- added C25: C_Small, Capacitor_SMD:C_0805_2012Metric_Pad1.18x1.45mm_HandSolder, F.Cu at (193.3, 92.4)
- added C35: C_Small, Capacitor_SMD:C_0805_2012Metric_Pad1.18x1.45mm_HandSolder, F.Cu at (193.3, 73.3)
- added C36: C_Small, Capacitor_SMD:C_0805_2012Metric_Pad1.18x1.45mm_HandSolder, F.Cu at (231.0, 82.9)
- added C46: C_Small, Capacitor_SMD:C_0805_2012Metric_Pad1.18x1.45mm_HandSolder, F.Cu at (212.0, 82.9)
- added C55: C_Small, Capacitor_SMD:C_0805_2012Metric_Pad1.18x1.45mm_HandSolder, F.Cu at (193.3, 54.3)
- added C56: C_Small, Capacitor_SMD:C_0805_2012Metric_Pad1.18x1.45mm_HandSolder, F.Cu at (212.3, 54.3)
- added C65: C_Small, Capacitor_SMD:C_0805_2012Metric_Pad1.18x1.45mm_HandSolder, B.Cu at (200.8, 82.9)
- added C66: C_Small, Capacitor_SMD:C_0805_2012Metric_Pad1.18x1.45mm_HandSolder, B.Cu at (181.3, 92.4)
- added C75: C_Small, Capacitor_SMD:C_0805_2012Metric_Pad1.18x1.45mm_HandSolder, B.Cu at (219.5, 82.9)
- added C85: C_Small, Capacitor_SMD:C_0805_2012Metric_Pad1.18x1.45mm_HandSolder, B.Cu at (200.4, 54.3)
- added C86: C_Small, Capacitor_SMD:C_0805_2012Metric_Pad1.18x1.45mm_HandSolder, B.Cu at (181.3, 73.3)
- added C96: C_Small, Capacitor_SMD:C_0805_2012Metric_Pad1.18x1.45mm_HandSolder, B.Cu at (181.3, 54.3)
- added J2: Conn_01x10, Connector_PinHeader_2.54mm:PinHeader_1x10_P2.54mm_Vertical, F.Cu at (182.4, 20.5)
- added LED25: MX_SK6812MINI-E, PCM_marbastlib-mx:LED_MX_6028R, F.Cu at (187.3, 92.4)
- added LED35: MX_SK6812MINI-E, PCM_marbastlib-mx:LED_MX_6028R, F.Cu at (187.3, 73.3)
- added LED36: MX_SK6812MINI-E, PCM_marbastlib-mx:LED_MX_6028R, F.Cu at (225.4, 82.9)
- added LED46: MX_SK6812MINI-E, PCM_marbastlib-mx:LED_MX_6028R, F.Cu at (206.4, 82.9)
- added LED55: MX_SK6812MINI-E, PCM_marbastlib-mx:LED_MX_6028R, F.Cu at (187.3, 54.3)
- added LED56: MX_SK6812MINI-E, PCM_marbastlib-mx:LED_MX_6028R, F.Cu at (206.4, 54.3)
- added LED65: MX_SK6812MINI-E, PCM_marbastlib-mx:LED_MX_6028R, B.Cu at (225.4, 82.9)
- added LED66: MX_SK6812MINI-E, PCM_marbastlib-mx:LED_MX_6028R, B.Cu at (187.3, 92.4)
- added LED75: MX_SK6812MINI-E, PCM_marbastlib-mx:LED_MX_6028R, B.Cu at (206.4, 82.9)
- added LED85: MX_SK6812MINI-E, PCM_marbastlib-mx:LED_MX_6028R, B.Cu at (206.4, 54.3)
- added LED86: MX_SK6812MINI-E, PCM_marbastlib-mx:LED_MX_6028R, B.Cu at (187.3, 73.3)
- added LED96: MX_SK6812MINI-E, PCM_marbastlib-mx:LED_MX_6028R, B.Cu at (187.3, 54.3)
- D25: renamed from D6; footprint keyboard_parts:D_SOD123W_hand -> Diode_SMD:D_SOD-323_HandSoldering
- D35: renamed from D5; footprint keyboard_parts:D_SOD123W_hand -> Diode_SMD:D_SOD-323_HandSoldering
- D36: renamed from D3; footprint keyboard_parts:D_SOD123W_hand -> Diode_SMD:D_SOD-323_HandSoldering
- D46: renamed from D2; footprint keyboard_parts:D_SOD123W_hand -> Diode_SMD:D_SOD-323_HandSoldering
- D55: renamed from D4; footprint keyboard_parts:D_SOD123W_hand -> Diode_SMD:D_SOD-323_HandSoldering
- D56: renamed from D1; footprint keyboard_parts:D_SOD123W_hand -> Diode_SMD:D_SOD-323_HandSoldering
- D65: renamed from D12; footprint keyboard_parts:D_SOD123W_hand -> Diode_SMD:D_SOD-323_HandSoldering
- D66: renamed from D9; footprint keyboard_parts:D_SOD123W_hand -> Diode_SMD:D_SOD-323_HandSoldering
- D75: renamed from D11; footprint keyboard_parts:D_SOD123W_hand -> Diode_SMD:D_SOD-323_HandSoldering
- D85: renamed from D10; footprint keyboard_parts:D_SOD123W_hand -> Diode_SMD:D_SOD-323_HandSoldering
- D86: renamed from D8; footprint keyboard_parts:D_SOD123W_hand -> Diode_SMD:D_SOD-323_HandSoldering
- D96: renamed from D7; footprint keyboard_parts:D_SOD123W_hand -> Diode_SMD:D_SOD-323_HandSoldering
- moved D56 12.8 mm to (206.4, 41.2)
- moved D65 12.8 mm to (225.5, 69.8)
- moved D25 12.8 mm to (187.3, 79.3)
- moved D35 12.8 mm to (187.3, 60.3)
- moved D36 12.8 mm to (225.4, 69.8)
- moved D46 12.8 mm to (206.4, 69.8)
- moved D55 12.8 mm to (187.3, 41.2)
- moved D66 12.8 mm to (187.3, 79.3)
- moved D75 12.8 mm to (206.4, 69.8)
- moved D85 12.8 mm to (206.4, 41.2)
- moved D96 12.8 mm to (187.3, 41.2)
- moved D86 11.8 mm to (187.3, 61.3)
- moved MX55 0.07 mm to (187.3, 49.3)
Connections:
- J1 pad 10: unconnected-(J1-Pin_10-Pad10) -> /VDD
- J1 pad 6: unconnected-(J1-Pin_6-Pad6) -> /DIN_L
- J1 pad 7: unconnected-(J1-Pin_7-Pad7) -> /DOUT_L
- J1 pad 9: unconnected-(J1-Pin_9-Pad9) -> GND
Routing:
- net /ROW_3: track 116.5 -> 0.00 mm, vias 3 -> 0
- net /ROW_6: track 112.8 -> 0.00 mm, vias 1 -> 0
- net /COL_L6: track 87.8 -> 0.00 mm
- net /ROW_4: track 81.9 -> 0.00 mm, vias 3 -> 0
- net /ROW_2: track 71.2 -> 0.00 mm, vias 2 -> 0
- net /ROW_8: track 69.9 -> 0.00 mm, vias 1 -> 0
- net /COL_R5: track 69.1 -> 0.00 mm, vias 1 -> 0
- net /ROW_7: track 62.0 -> 0.00 mm, vias 1 -> 0
- net /COL_R6: track 59.3 -> 0.00 mm, vias 1 -> 0
- net /COL_L5: track 55.9 -> 0.00 mm, vias 1 -> 0
- net /ROW_5: track 50.4 -> 0.00 mm, vias 2 -> 0
- net /ROW_9: track 35.1 -> 0.00 mm, vias 1 -> 0
- net Net-(D86-A): track 10.2 -> 0.00 mm
- net Net-(D35-A): track 10.2 -> 0.00 mm
- net Net-(D96-A): track 10.2 -> 0.00 mm
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- removed copper zone on B.Cu, net /ROW_4
- removed copper zone on F.Cu, net /ROW_4

Commit message: Checkpoint - routing
Parts:
- moved J2 4.76 mm to (177.9, 18.7)
- moved D86 1.00 mm to (187.3, 60.3)
Routing:
- net /VDD: track 0.00 -> 212.5 mm, vias 0 -> 9
- net /COL_L6: track 0.00 -> 95.7 mm
- net /ROW_3: track 0.00 -> 75.7 mm, vias 0 -> 1
- net /ROW_4: track 0.00 -> 71.3 mm, vias 0 -> 1
- net /COL_L5: track 0.00 -> 66.0 mm
- net Net-(LED25-DIN): track 0.00 -> 64.6 mm
- net /ROW_2: track 0.00 -> 61.8 mm
- net Net-(LED65-DIN): track 0.00 -> 60.4 mm
- net /COL_R5: track 0.00 -> 59.0 mm, vias 0 -> 1
- net /COL_R6: track 0.00 -> 48.9 mm
- net Net-(LED75-DOUT): track 0.00 -> 47.0 mm
- net Net-(LED25-DOUT): track 0.00 -> 44.8 mm, vias 0 -> 2
- net Net-(LED46-DIN): track 0.00 -> 40.3 mm, vias 0 -> 2
- net /ROW_5: track 0.00 -> 33.4 mm
- net /DOUT_L: track 0.00 -> 31.8 mm, vias 0 -> 1
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
Commit message: SOD123 Diodes
Parts:
- D25, D35, D36, D46, D55, D56, D65, D66, D75, D85, D86, D96: footprint Diode_SMD:D_SOD-323_HandSoldering -> Diode_SMD:D_SOD-123F
- moved J2 10.0 mm to (177.9, 28.7)
Routing:
- net /ROW_8: track 0.00 -> 21.2 mm

Commit message: Routed
Parts:
- moved J2 3.44 mm to (179.1, 25.5)
Routing:
- net GND: track 19.8 -> 215.0 mm, vias 6 -> 22
- net /ROW_6: track 0.00 -> 105.4 mm, vias 0 -> 3
- net /ROW_7: track 0.00 -> 65.3 mm, vias 0 -> 1
- net /DOUT_R: track 0.00 -> 57.3 mm, vias 0 -> 5
- net /ROW_8: track 21.2 -> 60.1 mm, vias 0 -> 2
- net Net-(LED35-DOUT): track 0.00 -> 35.4 mm, vias 0 -> 2
- net /DIN_R: track 0.00 -> 32.9 mm, vias 0 -> 2
- net /COL_R5: track 59.0 -> 84.2 mm
- net /COL_R6: track 48.9 -> 69.5 mm, vias 0 -> 1
- net /ROW_9: track 0.00 -> 13.2 mm, vias 0 -> 1
- net /COL_L6: track 95.7 -> 97.4 mm
- net /VDD: track 212.5 -> 211.6 mm

Commit message: Fully routed
Parts:
- removed G*** (x2): LOGO, pillz:logo_sm
- removed J2: Conn_01x10, Connector_PinHeader_2.54mm:PinHeader_1x10_P2.54mm_Vertical
- C25, C35, C36, C46, C55, C56, C65, C66, C75, C85, C86, C96: value C_Small -> 0.1 µF
- D25, D35, D36, D46, D55, D56, D65, D66, D75, D85, D86, D96: footprint Diode_SMD:D_SOD-123F -> Diode_SMD:D_SOD-323_HandSoldering
Connections:
- D25 pad 1: /ROW_2 -> /DOUT_R
- D35 pad 1: /ROW_3 -> /COL_R5
- D36 pad 1: /ROW_3 -> /COL_R5
- D46 pad 1: /ROW_4 -> /DIN_R
- D65 pad 1: /ROW_6 -> /ROW_5
- D66 pad 1: /ROW_6 -> /ROW_5
- D75 pad 1: /ROW_7 -> /COL_L6
- D85 pad 1: /ROW_8 -> /COL_L5
- D86 pad 1: /ROW_8 -> /COL_L5
- D96 pad 1: /ROW_9 -> /DIN_L
- J1 pad 1: /ROW_4 -> /DIN_R
- J1 pad 2: /ROW_2 -> /DOUT_R
- J1 pad 7: /DOUT_L -> /COL_R6
- J1 pad 8: /ROW_3 -> /COL_R5
- LED55 pad 2: /DOUT_L -> /COL_R6
Routing:
- net /ROW_6: track 105.4 -> 0.00 mm, vias 3 -> 0
- net /ROW_5: track 33.4 -> 135.1 mm, vias 0 -> 3
- net /ROW_3: track 75.4 -> 0.00 mm, vias 1 -> 0
- net /ROW_4: track 71.3 -> 0.00 mm, vias 1 -> 0
- net /DIN_R: track 32.9 -> 101.7 mm, vias 2 -> 3
- net /COL_R5: track 84.2 -> 152.7 mm, vias 1 -> 2
- net /ROW_7: track 65.3 -> 0.00 mm, vias 1 -> 0
- net /COL_L6: track 97.4 -> 162.6 mm, vias 0 -> 1
- net /ROW_2: track 61.8 -> 0.00 mm
- net /ROW_8: track 60.1 -> 0.00 mm, vias 2 -> 0
- net /DOUT_R: track 57.3 -> 116.3 mm, vias 5 -> 4
- net /COL_L5: track 66.0 -> 119.1 mm, vias 0 -> 2
- net /DOUT_L: track 31.8 -> 0.00 mm, vias 1 -> 0
- net /COL_R6: track 69.5 -> 97.6 mm, vias 1 -> 2
- net /ROW_9: track 13.2 -> 0.00 mm, vias 1 -> 0
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Other:
- board text removed: "Pillz Mod thumb cluster LEFT Rev 2 github.com/dcpedit/pillzmod"
- board text removed: "Pillz Mod thumb cluster RIGHT Rev 2 github.com/dcpedit/pillzmod"

Commit message: checkpoint
Routing:
- net GND: track 222.6 -> 342.1 mm, vias 23 -> 29
- added copper zone on B.Cu, net GND
- added copper zone on F.Cu, net GND
